File: neptune-flight-computer/power.kicad_sch (KiCad schematic)
At the start: 32 parts

Commit message: Continued work on board
Parts:
- C? (x2): value (none) -> 0.1u; footprint (none) -> Capacitor_SMD:C_0402_1005Metric
- C?: value (none) -> 0.1u
- C?: value (none) -> 2.2u; footprint (none) -> Capacitor_SMD:C_0402_1005Metric
- C?: value (none) -> 1u
- U?: value (none) -> AP2210N-3.3TRG1; footprint (none) -> Package_TO_SOT_SMD:SOT-23
- U?: value (none) -> TPS54331D; footprint (none) -> Package_SO:SOIC-8-1EP_3.9x4.9mm_P1.27mm_EP2.29x3mm_ThermalVias
Changed lines of the file:
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@@
     (in_bom yes) (on_board yes) (fields_autoplaced)
     (property "Reference" "U?" (id 0) (at 158.115 71.12 0))
-    (property "Value" "" (id 1) (at 158.115 73.66 0))
-    (property "Footprint" "" (id 2) (at 158.115 81.28 0)
+    (property "Value" "AP2210N-3.3TRG1" (id 1) (at 158.115 73.66 0))
+    (property "Footprint" "Package_TO_SOT_SMD:SOT-23" (id 2) (at 158.115 81.28 0)
       (effects (font (size 1.27 1.27)) (justify bottom) hide)
     )
@@
       (effects (font (size 1.27 1.27)) (justify right))
     )
-    (property "Value" "" (id 1) (at 144.145 86.3662 0)
-      (effects (font (size 1.27 1.27)) (justify right))
-    )
-    (property "Footprint" "" (id 2) (at 140.97 85.09 0)
+    (property "Value" "0.1u" (id 1) (at 144.145 86.3662 0)
+      (effects (font (size 1.27 1.27)) (justify right))
+    )
+    (property "Footprint" "Capacitor_SMD:C_0402_1005Metric" (id 2) (at 140.97 85.09 0)
       (effects (font (size 1.27 1.27)) hide)
     )
@@
       (effects (font (size 1.27 1.27)) (justify left))
     )
-    (property "Value" "" (id 1) (at 189.23 31.7562 0)
+    (property "Value" "0.1u" (id 1) (at 189.23 31.7562 0)
       (effects (font (size 1.27 1.27)) (justify left))
     )
@@
       (effects (font (size 1.27 1.27)) (justify right))
     )
-    (property "Value" "" (id 1) (at 88.9 87.63 0)
-      (effects (font (size 1.27 1.27)) (justify right))
-    )
-    (property "Footprint" "" (id 2) (at 95.25 86.36 0)
+    (property "Value" "0.1u" (id 1) (at 88.9 87.63 0)
+      (effects (font (size 1.27 1.27)) (justify right))
+    )
+    (property "Footprint" "Capacitor_SMD:C_0402_1005Metric" (id 2) (at 95.25 86.36 0)
       (effects (font (size 1.27 1.27)) hide)
     )
@@
       (effects (font (size 1.27 1.27)) (justify right))
     )
-    (property "Value" "" (id 1) (at 184.15 86.3662 0)
-      (effects (font (size 1.27 1.27)) (justify right))
-    )
-    (property "Footprint" "" (id 2) (at 181.61 85.09 0)
+    (property "Value" "2.2u" (id 1) (at 184.15 86.3662 0)
+      (effects (font (size 1.27 1.27)) (justify right))
+    )
+    (property "Footprint" "Capacitor_SMD:C_0402_1005Metric" (id 2) (at 181.61 85.09 0)
       (effects (font (size 1.27 1.27)) hide)
     )
@@
       (effects (font (size 1.27 1.27)) (justify right))
     )
-    (property "Value" "" (id 1) (at 134.62 86.3662 0)
+    (property "Value" "1u" (id 1) (at 134.62 86.3662 0)
       (effects (font (size 1.27 1.27)) (justify right))
     )
@@
       (effects (font (size 1.524 1.524)))
     )
-    (property "Value" "" (id 1) (at 167.64 31.623 0)
+    (property "Value" "TPS54331D" (id 1) (at 167.64 31.623 0)
       (effects (font (size 1.524 1.524)))
     )
-    (property "Footprint" "" (id 2) (at 168.91 30.734 0)
+    (property "Footprint" "Package_SO:SOIC-8-1EP_3.9x4.9mm_P1.27mm_EP2.29x3mm_ThermalVias" (id 2) (at 168.91 30.734 0)
       (effects (font (size 1.524 1.524)) hide)
     )

Commit message: Continued pcb work
Parts:
- removed C? (x3): 0.1u, Capacitor_SMD:C_0402_1005Metric, symbol Device:C_Small
- added C? (x3): 100nF, Capacitor_SMD:C_0603_1608Metric, symbol Device:C_Small
Connections:
- net +5V: now also C?.1
- net GND: now also C?.2, C?.2
- net VDC: now also C?.1
- net at U?.1 (BOOT): now also C?.1
- net at D?.1 (K), L?.1, U?.8 (PH): now also C?.2
