File: neptune-flight-computer/power.kicad_sch (KiCad schematic)
At the start: 31 parts, among them J2 Conn_01x02, Q1 Si2301-TP, Q2 AO3401A, U1 ADR5040ARTZ-2.048, U2 LM393, U3 TPS54331D, U4 AP2210N-3.3TRG1

Commit message: Created production files
Parts:
- C16: value 2.2u -> 1u
- U4: value AP2210N-3.3TRG1 -> LP3993-33B3F; LCSC C155508 -> C387705
Changed lines of the file:
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@@
   (symbol (lib_id "AP2210N-3.3TRG1:AP2210N-3.3TRG1") (at 158.115 81.28 0) (unit 1)
     (in_bom yes) (on_board yes) (dnp no) (fields_autoplaced)
-    (property "Reference" "U4" (at 158.115 71.12 0)
-      (effects (font (size 1.27 1.27)))
-    )
-    (property "Value" "AP2210N-3.3TRG1" (at 158.115 73.66 0)
+    (property "Reference" "U4" (at 158.115 72.39 0)
+      (effects (font (size 1.27 1.27)))
+    )
+    (property "Value" "LP3993-33B3F" (at 158.115 74.93 0)
       (effects (font (size 1.27 1.27)))
     )
@@
       (effects (font (size 1.27 1.27)) (justify bottom) hide)
     )
-    (property "Datasheet" "https://datasheet.lcsc.com/lcsc/1810171025_Diodes-Incorporated-AP2210N-3-3TRG1_C155508.pdf" (at 158.115 81.28 0)
-      (effects (font (size 1.27 1.27)) hide)
-    )
-    (property "LCSC" "C155508" (at 158.115 81.28 0)
+    (property "Datasheet" "https://jlcpcb.com/partdetail/Lowpower-LP399333B3F/C387705" (at 158.115 81.28 0)
+      (effects (font (size 1.27 1.27)) hide)
+    )
+    (property "LCSC" "C387705" (at 158.115 81.28 0)
       (effects (font (size 1.27 1.27)) (justify bottom) hide)
     )
@@
       (effects (font (size 1.27 1.27)) (justify right))
     )
-    (property "Value" "2.2u" (at 184.15 86.3662 0)
+    (property "Value" "1u" (at 184.15 86.3662 0)
       (effects (font (size 1.27 1.27)) (justify right))
     )
