File: neptune-flight-computer/Sensors.kicad_sch (KiCad schematic)
At the start: 3 parts

Commit message: Added oscillator, setup sensor SPI
Connections:
- net +3V3: no longer U?.7 (PS)
- net GND: now also U?.7 (PS); no longer U?.12 (SDO2), U?.17 (SDO1), U?.20 (CSB3)
- net CE_ACC: now reaches U?.16 (CSB1)
- net CE_GYR: now reaches U?.5 (CSB2)
- net BMX_Int_1: no longer names the net of U?.19 (INT1)
- net SCL renamed IMU_SCK
- net SDA renamed IMU_MOSI
- new net CE_MAG: U?.20 (CSB3)
- new net IMU_MISO: U?.12 (SDO2), U?.17 (SDO1)
- no-connect marks 7 -> 6
Other:
- note added: "Tied low for SPI interface selection"
- note removed: "Tied high for I2C interface selection"
Changed lines of the file:
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@@
 (kicad_sch (version 20211123) (generator eeschema)
   (paper "A4")
-  (junction (at 32.385 62.23) (diameter 0) (color 0 0 0 0)
+  (junction (at 35.56 60.96) (diameter 0) (color 0 0 0 0)
   )
   (junction (at 81.28 76.2) (diameter 0) (color 0 0 0 0)
@@
   (junction (at 54.61 30.48) (diameter 0) (color 0 0 0 0)
   )
-  (junction (at 57.15 30.48) (diameter 0) (color 0 0 0 0)
-  )
   (junction (at 54.61 68.58) (diameter 0) (color 0 0 0 0)
   )
   (junction (at 81.28 86.36) (diameter 0) (color 0 0 0 0)
   )
-  (no_connect (at 36.83 36.83))
+  (no_connect (at 72.39 41.91))
   (no_connect (at 72.39 59.69))
   (no_connect (at 72.39 46.99))
@@
   (no_connect (at 72.39 52.07))
   (no_connect (at 72.39 44.45))
-  (no_connect (at 36.83 39.37))
   (wire (pts (xy 52.07 31.75) (xy 52.07 30.48))
     (stroke (width 0) (type default) (color 0 0 0 0))
@@
     (stroke (width 0) (type default) (color 0 0 0 0))
   )
+  (wire (pts (xy 33.02 36.83) (xy 36.83 36.83))
+    (stroke (width 0) (type default) (color 0 0 0 0))
+  )
   (wire (pts (xy 57.15 68.58) (xy 54.61 68.58))
     (stroke (width 0) (type default) (color 0 0 0 0))
   )
+  (wire (pts (xy 35.56 62.23) (xy 36.83 62.23))
+    (stroke (width 0) (type default) (color 0 0 0 0))
+  )
   (wire (pts (xy 57.15 67.31) (xy 57.15 68.58))
     (stroke (width 0) (type default) (color 0 0 0 0))
   )
+  (wire (pts (xy 33.02 39.37) (xy 36.83 39.37))
+    (stroke (width 0) (type default) (color 0 0 0 0))
+  )
   (wire (pts (xy 87.63 76.2) (xy 87.63 78.74))
     (stroke (width 0) (type default) (color 0 0 0 0))
@@
     (stroke (width 0) (type default) (color 0 0 0 0))
   )
-  (wire (pts (xy 72.39 30.48) (xy 72.39 36.83))
+  (wire (pts (xy 35.56 60.96) (xy 35.56 62.23))
     (stroke (width 0) (type default) (color 0 0 0 0))
   )
@@
     (stroke (width 0) (type default) (color 0 0 0 0))
   )
-  (wire (pts (xy 32.385 52.07) (xy 36.83 52.07))
+  (wire (pts (xy 33.02 52.07) (xy 36.83 52.07))
     (stroke (width 0) (type default) (color 0 0 0 0))
   )
@@
     (stroke (width 0) (type default) (color 0 0 0 0))
   )
-  (wire (pts (xy 31.75 41.91) (xy 36.83 41.91))
+  (wire (pts (xy 33.02 41.91) (xy 36.83 41.91))
     (stroke (width 0) (type default) (color 0 0 0 0))
   )
@@
     (stroke (width 0) (type default) (color 0 0 0 0))
   )
-  (wire (pts (xy 32.385 59.69) (xy 32.385 62.23))
-    (stroke (width 0) (type default) (color 0 0 0 0))
-  )
-  (wire (pts (xy 32.385 49.53) (xy 36.83 49.53))
+  (wire (pts (xy 33.02 49.53) (xy 36.83 49.53))
     (stroke (width 0) (type default) (color 0 0 0 0))
   )
@@
     (stroke (width 0) (type default) (color 0 0 0 0))
   )
-  (wire (pts (xy 72.39 41.91) (xy 77.47 41.91))
-    (stroke (width 0) (type default) (color 0 0 0 0))
-  )
-  (wire (pts (xy 57.15 30.48) (xy 72.39 30.48))
-    (stroke (width 0) (type default) (color 0 0 0 0))
-  )
-  (wire (pts (xy 36.83 59.69) (xy 32.385 59.69))
+  (wire (pts (xy 35.56 59.69) (xy 36.83 59.69))
+    (stroke (width 0) (type default) (color 0 0 0 0))
+  )
+  (wire (pts (xy 33.02 60.96) (xy 35.56 60.96))
     (stroke (width 0) (type default) (color 0 0 0 0))
   )
@@
     (stroke (width 0) (type default) (color 0 0 0 0))
   )
-  (wire (pts (xy 32.385 62.23) (xy 36.83 62.23))
-    (stroke (width 0) (type default) (color 0 0 0 0))
-  )
-  (text "Place orientation \nmarking on PCB" (at 100.965 54.61 0)
+  (wire (pts (xy 35.56 60.96) (xy 35.56 59.69))
+    (stroke (width 0) (type default) (color 0 0 0 0))
+  )
+  (text "Place orientation \nmarking on PCB" (at 81.28 21.59 0)
     (effects (font (size 1.27 1.27)) (justify left bottom))
   )
-  (text "Tied high for I2C\ninterface selection" (at 60.96 29.21 0)
+  (text "Tied low for SPI\ninterface selection" (at 72.39 35.56 0)
     (effects (font (size 0.8 0.8)) (justify left bottom))
   )
@@
     (effects (font (size 3.9878 3.9878)) (justify left bottom))
   )
-  (hierarchical_label "SDA" (shape input) (at 32.385 49.53 180)
-    (effects (font (size 1.27 1.27)) (justify right))
-  )
-  (hierarchical_label "BMX_Int_1" (shape input) (at 77.47 41.91 0)
-    (effects (font (size 1.27 1.27)) (justify left))
-  )
-  (hierarchical_label "SCL" (shape input) (at 32.385 52.07 180)
-    (effects (font (size 1.27 1.27)) (justify right))
+  (hierarchical_label "IMU_MISO" (shape output) (at 33.02 60.96 180)
+    (effects (font (size 1.27 1.27)) (justify right))
+  )
+  (hierarchical_label "CE_GYR" (shape input) (at 33.02 39.37 180)
+    (effects (font (size 1.27 1.27)) (justify right))
+  )
+  (hierarchical_label "IMU_MOSI" (shape input) (at 33.02 49.53 180)
+    (effects (font (size 1.27 1.27)) (justify right))
+  )
+  (hierarchical_label "CE_MAG" (shape input) (at 33.02 41.91 180)
+    (effects (font (size 1.27 1.27)) (justify right))
+  )
+  (hierarchical_label "IMU_SCK" (shape input) (at 33.02 52.07 180)
+    (effects (font (size 1.27 1.27)) (justify right))
+  )
+  (hierarchical_label "CE_ACC" (shape input) (at 33.02 36.83 180)
+    (effects (font (size 1.27 1.27)) (justify right))
+  )
+  (symbol (lib_id "power:GND") (at 72.39 36.83 0) (unit 1)
+    (in_bom yes) (on_board yes)
+    (property "Reference" "#PWR?" (id 0) (at 72.39 43.18 0)
+      (effects (font (size 1.27 1.27)) hide)
+    )
+    (property "Value" "" (id 1) (at 76.2 38.1 0))
+    (property "Footprint" "" (id 2) (at 72.39 36.83 0)
+      (effects (font (size 1.27 1.27)) hide)
+    )
+    (property "Datasheet" "" (id 3) (at 72.39 36.83 0)
+      (effects (font (size 1.27 1.27)) hide)
+    )
+    (pin "1")
   )
   (symbol (lib_id "power:+3.3V") (at 81.28 76.2 0) (unit 1)
@@
     (pin "9")
   )
-  (symbol (lib_id "power:GND") (at 32.385 62.23 0) (unit 1)
-    (in_bom yes) (on_board yes)
-    (property "Reference" "#PWR?" (id 0) (at 32.385 68.58 0)
-      (effects (font (size 1.27 1.27)) hide)
-    )
-    (property "Value" "GND" (id 1) (at 32.512 66.6242 0))
-    (property "Footprint" "" (id 2) (at 32.385 62.23 0)
-      (effects (font (size 1.27 1.27)) hide)
-    )
-    (property "Datasheet" "" (id 3) (at 32.385 62.23 0)
-      (effects (font (size 1.27 1.27)) hide)
-    )
-    (pin "1")
-  )
   (symbol (lib_id "power:GND") (at 81.28 86.36 0) (unit 1)
     (in_bom yes) (on_board yes)
@@
       (effects (font (size 1.27 1.27)) hide)
     )
-    (property "Value" "" (id 1) (at 54.61 25.4 0))
+    (property "Value" "+3.3V" (id 1) (at 54.61 25.4 0))
     (property "Footprint" "" (id 2) (at 54.61 30.48 0)
       (effects (font (size 1.27 1.27)) hide)
@@
       (effects (font (size 1.27 1.27)) hide)
     )
-    (pin "1")
-  )
-  (symbol (lib_id "power:GND") (at 31.75 41.91 0) (unit 1)
-    (in_bom yes) (on_board yes)
-    (property "Reference" "#PWR?" (id 0) (at 31.75 48.26 0)
-      (effects (font (size 1.27 1.27)) hide)
-    )
-    (property "Value" "GND" (id 1) (at 31.877 46.3042 0))
-    (property "Footprint" "" (id 2) (at 31.75 41.91 0)
-      (effects (font (size 1.27 1.27)) hide)
-    )
-    (property "Datasheet" "" (id 3) (at 31.75 41.91 0)
-      (effects (font (size 1.27 1.27)) hide)
-    )

Commit message: Schematic done I think
Parts:
- U8: renamed from U?; footprint Local_footprints:BMX055 -> Local Library:BMX055
- gave numbers to parts that had none: 2
Changed lines of the file:
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@@
   (symbol (lib_id "power:GND") (at 72.39 36.83 0) (unit 1)
     (in_bom yes) (on_board yes) (dnp no)
-    (property "Reference" "#PWR?" (at 72.39 43.18 0)
+    (property "Reference" "#PWR061" (at 72.39 43.18 0)
       (effects (font (size 1.27 1.27)) hide)
     )
@@
       (project "neptune"
         (path "/e63e39d7-6ac0-4ffd-8aa3-1841a4541b55/fd0daead-056b-49b0-b136-e76d44737a4c"
-          (reference "#PWR?") (unit 1)
+          (reference "#PWR061") (unit 1)
         )
       )
@@
   (symbol (lib_id "power:+3.3V") (at 81.28 76.2 0) (unit 1)
     (in_bom yes) (on_board yes) (dnp no) (fields_autoplaced)
-    (property "Reference" "#PWR?" (at 81.28 80.01 0)
+    (property "Reference" "#PWR062" (at 81.28 80.01 0)
       (effects (font (size 1.27 1.27)) hide)
     )
@@
       (project "neptune"
         (path "/e63e39d7-6ac0-4ffd-8aa3-1841a4541b55/fd0daead-056b-49b0-b136-e76d44737a4c"
-          (reference "#PWR?") (unit 1)
+          (reference "#PWR062") (unit 1)
         )
       )
@@
   (symbol (lib_id "BMX055:BMX055") (at 54.61 49.53 0) (unit 1)
     (in_bom yes) (on_board yes) (dnp no)
-    (property "Reference" "U?" (at 50.8 48.26 0)
+    (property "Reference" "U8" (at 50.8 48.26 0)
       (effects (font (size 1.27 1.27)) (justify left))
     )
@@
       (effects (font (size 1.27 1.27)) (justify left))
     )
-    (property "Footprint" "Local_footprints:BMX055" (at 54.61 49.53 0)
+    (property "Footprint" "Local Library:BMX055" (at 54.61 49.53 0)
       (effects (font (size 1.27 1.27)) (justify left bottom) hide)
     )
@@
       (project "neptune"
         (path "/e63e39d7-6ac0-4ffd-8aa3-1841a4541b55/fd0daead-056b-49b0-b136-e76d44737a4c"
-          (reference "U?") (unit 1)
+          (reference "U8") (unit 1)
         )
       )
@@
   (symbol (lib_id "power:GND") (at 81.28 86.36 0) (unit 1)
     (in_bom yes) (on_board yes) (dnp no)
-    (property "Reference" "#PWR?" (at 81.28 92.71 0)
+    (property "Reference" "#PWR063" (at 81.28 92.71 0)
       (effects (font (size 1.27 1.27)) hide)
     )
@@
       (project "neptune"
         (path "/e63e39d7-6ac0-4ffd-8aa3-1841a4541b55/fd0daead-056b-49b0-b136-e76d44737a4c"
-          (reference "#PWR?") (unit 1)
+          (reference "#PWR063") (unit 1)
         )
       )
@@
   (symbol (lib_id "power:+3.3V") (at 54.61 30.48 0) (unit 1)
     (in_bom yes) (on_board yes) (dnp no) (fields_autoplaced)
-    (property "Reference" "#PWR?" (at 54.61 34.29 0)
+    (property "Reference" "#PWR059" (at 54.61 34.29 0)
       (effects (font (size 1.27 1.27)) hide)
     )
@@
       (project "neptune"
         (path "/e63e39d7-6ac0-4ffd-8aa3-1841a4541b55/fd0daead-056b-49b0-b136-e76d44737a4c"
-          (reference "#PWR?") (unit 1)
+          (reference "#PWR059") (unit 1)
         )
       )
@@
   (symbol (lib_id "power:GND") (at 54.61 68.58 0) (unit 1)
     (in_bom yes) (on_board yes) (dnp no)
-    (property "Reference" "#PWR?" (at 54.61 74.93 0)
+    (property "Reference" "#PWR060" (at 54.61 74.93 0)
       (effects (font (size 1.27 1.27)) hide)
     )
@@
       (project "neptune"
         (path "/e63e39d7-6ac0-4ffd-8aa3-1841a4541b55/fd0daead-056b-49b0-b136-e76d44737a4c"
-          (reference "#PWR?") (unit 1)
+          (reference "#PWR060") (unit 1)
         )
       )
@@
   (symbol (lib_id "Device:C_Small") (at 87.63 81.28 0) (unit 1)
     (in_bom yes) (on_board yes) (dnp no)
-    (property "Reference" "C?" (at 90.17 78.74 0)
+    (property "Reference" "C25" (at 90.17 78.74 0)
       (effects (font (size 1.27 1.27)) (justify left))
     )
@@
       (project "neptune"
         (path "/e63e39d7-6ac0-4ffd-8aa3-1841a4541b55/fd0daead-056b-49b0-b136-e76d44737a4c"
-          (reference "C?") (unit 1)
+          (reference "C25") (unit 1)
         )
       )
@@
   (symbol (lib_id "Device:C_Small") (at 74.93 81.28 0) (unit 1)
     (in_bom yes) (on_board yes) (dnp no)
-    (property "Reference" "C?" (at 77.47 78.74 0)
+    (property "Reference" "C24" (at 77.47 78.74 0)
       (effects (font (size 1.27 1.27)) (justify left))
     )
@@
       (project "neptune"
         (path "/e63e39d7-6ac0-4ffd-8aa3-1841a4541b55/fd0daead-056b-49b0-b136-e76d44737a4c"
-          (reference "C?") (unit 1)
-        )
-      )
+          (reference "C24") (unit 1)
+        )
+      )
