File: neptune-flight-computer/data_management.kicad_sch (KiCad schematic)
At the start: 4 parts

Commit message: Continued work on board
Parts:
- C?: value 10uF -> (none); footprint Capacitor_SMD:C_0603_1608Metric -> (none)
- C?: value 100nF -> (none); footprint Capacitor_SMD:C_0603_1608Metric -> (none)
- J?: value Conn_Coaxial -> (none); footprint Connector_Coaxial:SMA_Amphenol_132291_Vertical -> (none)
- U?: value RFM95W-915S2 -> (none); footprint RF_Module:HOPERF_RFM9XW_SMD -> (none)
Other:
- note added: "Data transmission"
Changed lines of the file:
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@@
     (effects (font (size 1.27 1.27)) (justify left bottom))
   )
-  (text "RFM95W" (at 40.64 36.83 0)
-    (effects (font (size 3.9878 3.9878)) (justify left bottom))
+  (text "RFM95W" (at 20.32 41.91 0)
+    (effects (font (size 1.27 1.27) (thickness 0.254) bold) (justify left bottom))
+  )
+  (text "Data transmission" (at 19.05 35.56 0)
+    (effects (font (size 2.3 2.3) italic) (justify left bottom))
   )
   (hierarchical_label "RESET_RF" (shape input) (at 34.29 76.2 180)
@@
       (effects (font (size 1.27 1.27)) hide)
     )
-    (property "Value" "GND" (id 1) (at 49.657 94.5642 0))
+    (property "Value" "" (id 1) (at 49.657 94.5642 0))
     (property "Footprint" "" (id 2) (at 49.53 90.17 0)
       (effects (font (size 1.27 1.27)) hide)
@@
       (effects (font (size 1.27 1.27)) hide)
     )
-    (property "Value" "GND" (id 1) (at 73.787 74.2442 0))
+    (property "Value" "" (id 1) (at 73.787 74.2442 0))
     (property "Footprint" "" (id 2) (at 73.66 69.85 0)
       (effects (font (size 1.27 1.27)) hide)
@@
       (effects (font (size 1.27 1.27)) (justify left))
     )
-    (property "Value" "Conn_Coaxial" (id 1) (at 76.2 66.4464 0)
+    (property "Value" "" (id 1) (at 76.2 66.4464 0)
       (effects (font (size 1.27 1.27)) (justify left))
     )
-    (property "Footprint" "Connector_Coaxial:SMA_Amphenol_132291_Vertical" (id 2) (at 73.66 63.5 0)
+    (property "Footprint" "" (id 2) (at 73.66 63.5 0)
       (effects (font (size 1.27 1.27)) hide)
     )
@@
     (in_bom yes) (on_board yes)
     (property "Reference" "U?" (id 0) (at 39.37 53.34 0))
-    (property "Value" "RFM95W-915S2" (id 1) (at 39.37 55.88 0))
-    (property "Footprint" "RF_Module:HOPERF_RFM9XW_SMD" (id 2) (at -34.29 29.21 0)
+    (property "Value" "" (id 1) (at 39.37 55.88 0))
+    (property "Footprint" "" (id 2) (at -34.29 29.21 0)
       (effects (font (size 1.27 1.27)) hide)
     )
@@
       (effects (font (size 1.27 1.27)) hide)
     )
-    (property "Value" "VDD" (id 1) (at 49.911 42.5958 0))
+    (property "Value" "" (id 1) (at 49.911 42.5958 0))
     (property "Footprint" "" (id 2) (at 49.53 46.99 0)
       (effects (font (size 1.27 1.27)) hide)
@@
       (effects (font (size 1.27 1.27)) (justify left))
     )
-    (property "Value" "10uF" (id 1) (at 73.66 53.34 0)
+    (property "Value" "" (id 1) (at 73.66 53.34 0)
       (effects (font (size 1.27 1.27)) (justify left))
     )
-    (property "Footprint" "Capacitor_SMD:C_0603_1608Metric" (id 2) (at 71.12 53.34 0)
+    (property "Footprint" "" (id 2) (at 71.12 53.34 0)
       (effects (font (size 1.27 1.27)) hide)
     )
@@
       (effects (font (size 1.27 1.27)) (justify left))
     )
-    (property "Value" "100nF" (id 1) (at 62.23 53.34 0)
+    (property "Value" "" (id 1) (at 62.23 53.34 0)
       (effects (font (size 1.27 1.27)) (justify left))
     )
-    (property "Footprint" "Capacitor_SMD:C_0603_1608Metric" (id 2) (at 59.69 53.34 0)
+    (property "Footprint" "" (id 2) (at 59.69 53.34 0)
       (effects (font (size 1.27 1.27)) hide)
     )
@@
       (effects (font (size 1.27 1.27)) hide)
     )
-    (property "Value" "GND" (id 1) (at 66.167 61.5442 0))
+    (property "Value" "" (id 1) (at 66.167 61.5442 0))
     (property "Footprint" "" (id 2) (at 66.04 57.15 0)
       (effects (font (size 1.27 1.27)) hide)

Commit message: Added oscillator, setup sensor SPI
Parts:
- C?: value (none) -> 10uF; footprint (none) -> Capacitor_SMD:C_0603_1608Metric
- C?: value (none) -> 100nF; footprint (none) -> Capacitor_SMD:C_0603_1608Metric
- J?: value (none) -> Conn_Coaxial; footprint (none) -> Connector_Coaxial:SMA_Amphenol_132291_Vertical
- U?: value (none) -> RFM95W-915S2; footprint (none) -> RF_Module:HOPERF_RFM9XW_SMD
Changed lines of the file:
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@@
       (effects (font (size 1.27 1.27)) hide)
     )
-    (property "Value" "" (id 1) (at 49.657 94.5642 0))
+    (property "Value" "GND" (id 1) (at 49.657 94.5642 0))
     (property "Footprint" "" (id 2) (at 49.53 90.17 0)
       (effects (font (size 1.27 1.27)) hide)
@@
       (effects (font (size 1.27 1.27)) hide)
     )
-    (property "Value" "" (id 1) (at 73.787 74.2442 0))
+    (property "Value" "GND" (id 1) (at 73.787 74.2442 0))
     (property "Footprint" "" (id 2) (at 73.66 69.85 0)
       (effects (font (size 1.27 1.27)) hide)
@@
       (effects (font (size 1.27 1.27)) (justify left))
     )
-    (property "Value" "" (id 1) (at 76.2 66.4464 0)
+    (property "Value" "Conn_Coaxial" (id 1) (at 76.2 66.4464 0)
       (effects (font (size 1.27 1.27)) (justify left))
     )
-    (property "Footprint" "" (id 2) (at 73.66 63.5 0)
+    (property "Footprint" "Connector_Coaxial:SMA_Amphenol_132291_Vertical" (id 2) (at 73.66 63.5 0)
       (effects (font (size 1.27 1.27)) hide)
     )
@@
     (in_bom yes) (on_board yes)
     (property "Reference" "U?" (id 0) (at 39.37 53.34 0))
-    (property "Value" "" (id 1) (at 39.37 55.88 0))
-    (property "Footprint" "" (id 2) (at -34.29 29.21 0)
+    (property "Value" "RFM95W-915S2" (id 1) (at 39.37 55.88 0))
+    (property "Footprint" "RF_Module:HOPERF_RFM9XW_SMD" (id 2) (at -34.29 29.21 0)
       (effects (font (size 1.27 1.27)) hide)
     )
@@
       (effects (font (size 1.27 1.27)) hide)
     )
-    (property "Value" "" (id 1) (at 49.911 42.5958 0))
+    (property "Value" "VDD" (id 1) (at 49.911 42.5958 0))
     (property "Footprint" "" (id 2) (at 49.53 46.99 0)
       (effects (font (size 1.27 1.27)) hide)
@@
       (effects (font (size 1.27 1.27)) (justify left))
     )
-    (property "Value" "" (id 1) (at 73.66 53.34 0)
+    (property "Value" "10uF" (id 1) (at 73.66 53.34 0)
       (effects (font (size 1.27 1.27)) (justify left))
     )
-    (property "Footprint" "" (id 2) (at 71.12 53.34 0)
+    (property "Footprint" "Capacitor_SMD:C_0603_1608Metric" (id 2) (at 71.12 53.34 0)
       (effects (font (size 1.27 1.27)) hide)
     )
@@
       (effects (font (size 1.27 1.27)) (justify left))
     )
-    (property "Value" "" (id 1) (at 62.23 53.34 0)
+    (property "Value" "100nF" (id 1) (at 62.23 53.34 0)
       (effects (font (size 1.27 1.27)) (justify left))
     )
-    (property "Footprint" "" (id 2) (at 59.69 53.34 0)
+    (property "Footprint" "Capacitor_SMD:C_0603_1608Metric" (id 2) (at 59.69 53.34 0)
       (effects (font (size 1.27 1.27)) hide)
     )
@@
       (effects (font (size 1.27 1.27)) hide)
     )
-    (property "Value" "" (id 1) (at 66.167 61.5442 0))
+    (property "Value" "GND" (id 1) (at 66.167 61.5442 0))
     (property "Footprint" "" (id 2) (at 66.04 57.15 0)
       (effects (font (size 1.27 1.27)) hide)

Commit message: Continued pcb work
Parts:
- removed C?: 10uF, Capacitor_SMD:C_0603_1608Metric, symbol Device:C_Small
- removed C?: 100nF, Capacitor_SMD:C_0603_1608Metric, symbol Device:C_Small
- added C? (x2): 100nF, Capacitor_SMD:C_0603_1608Metric, symbol Device:C_Small
- added J7: THD2528-11SD-GF, Local_footprints:THD252811SDGF, symbol THD2528-11SD-GF:THD2528-11SD-GF
Connections:
- net GND: now also C?.2, C?.2, J7.6 (VSS), J7.MP1, J7.MP2, J7.MP3, J7.MP4
- net VDD renamed +3.3V
- net +3.3V: now also C?.1, C?.1, J7.4 (VDD)
- new net CLK_SD: J7.5 (CLX)
- new net CS_SD: J7.2 (CD/DAT3), J7.9 (CD)
- new net MISO_SD: J7.7 (DAT0)
- new net MOSI_SD: J7.3 (CMD)
- no-connect marks 5 -> 7
Other:
- note added: "Data storage"
- note added: "IC protection"
- note added: "SD card"
- moved on the sheet: J?, U?

Commit message: Schematic done I think
Parts:
- J7: footprint Local_footprints:THD252811SDGF -> Local Library:THD252811SDGF
- gave numbers to parts that had none: 2
Changed lines of the file:
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@@
   (symbol (lib_id "power:GND") (at 46.99 91.44 0) (unit 1)
     (in_bom yes) (on_board yes) (dnp no)
-    (property "Reference" "#PWR?" (at 46.99 97.79 0)
+    (property "Reference" "#PWR037" (at 46.99 97.79 0)
       (effects (font (size 1.27 1.27)) hide)
     )
@@
       (project "neptune"
         (path "/e63e39d7-6ac0-4ffd-8aa3-1841a4541b55/b694d9b6-8e2a-4217-a81b-e156ec88b46a"
-          (reference "#PWR?") (unit 1)
+          (reference "#PWR037") (unit 1)
         )
       )
@@
   (symbol (lib_id "power:GND") (at 66.04 71.12 0) (unit 1)
     (in_bom yes) (on_board yes) (dnp no)
-    (property "Reference" "#PWR?" (at 66.04 77.47 0)
+    (property "Reference" "#PWR038" (at 66.04 77.47 0)
       (effects (font (size 1.27 1.27)) hide)
     )
@@
       (project "neptune"
         (path "/e63e39d7-6ac0-4ffd-8aa3-1841a4541b55/b694d9b6-8e2a-4217-a81b-e156ec88b46a"
-          (reference "#PWR?") (unit 1)
+          (reference "#PWR038") (unit 1)
         )
       )
@@
       (effects (font (size 1.27 1.27)))
     )
-    (property "Footprint" "Local_footprints:THD252811SDGF" (at 153.67 48.26 0)
+    (property "Footprint" "Local Library:THD252811SDGF" (at 153.67 48.26 0)
       (effects (font (size 1.27 1.27)) (justify left) hide)
     )
@@
   (symbol (lib_id "Connector:Conn_Coaxial") (at 66.04 64.77 0) (unit 1)
     (in_bom yes) (on_board yes) (dnp no)
-    (property "Reference" "J?" (at 68.58 65.405 0)
+    (property "Reference" "J3" (at 68.58 65.405 0)
       (effects (font (size 1.27 1.27)) (justify left))
     )
@@
       (project "neptune"
         (path "/e63e39d7-6ac0-4ffd-8aa3-1841a4541b55/b694d9b6-8e2a-4217-a81b-e156ec88b46a"
-          (reference "J?") (unit 1)
+          (reference "J3") (unit 1)
         )
       )
@@
   (symbol (lib_id "RF_Module:RFM95W-915S2") (at 46.99 72.39 0) (unit 1)
     (in_bom yes) (on_board yes) (dnp no)
-    (property "Reference" "U?" (at 36.83 54.61 0)
+    (property "Reference" "U5" (at 36.83 54.61 0)
       (effects (font (size 1.27 1.27)))
     )
@@
       (project "neptune"
         (path "/e63e39d7-6ac0-4ffd-8aa3-1841a4541b55/b694d9b6-8e2a-4217-a81b-e156ec88b46a"
-          (reference "U?") (unit 1)
-        )
-      )
+          (reference "U5") (unit 1)
+        )
+      )
