File: neptune-flight-computer/STM32.kicad_sch (KiCad schematic)
At the start: 15 parts

Commit message: Added oscillator, setup sensor SPI
Parts:
- added C? (x2): 33p, Capacitor_SMD:C_0402_1005Metric, symbol Device:C_Small
- added J? (x2): Conn_01x04, Connector_PinHeader_2.54mm:PinHeader_1x04_P2.54mm_Vertical, symbol Connector_Generic:Conn_01x04
- added Y?: (no value), symbol Device:Crystal
- C?: value (none) -> 100n
- C?: value (none) -> 10n
- C?: value (none) -> 1u
- J?: value Conn_01x04 -> (none); footprint footprints:JST_SM04B-GHS-TB(LF)(SN)- -> (none)
- L?: value (none) -> 10u
Connections:
- net GND: now also C?.2, C?.2, J?.3 (Pin_3), J?.3 (Pin_3)
- net S1_feedback: now reaches U?.16 (PA2)
- net S1_feedback: now also J?.4 (Pin_4)
- net S2_feedback: now reaches U?.17 (PA3)
- net S2_feedback: now also J?.4 (Pin_4)
- net IMU_SCK: now reaches U?.21 (PA5)
- net IMU_MISO: now reaches U?.22 (PA6)
- net IMU_MOSI: now reaches U?.23 (PA7)
- net CE_ACC: now reaches U?.26 (PB0)
- net CE_GYR: now reaches U?.27 (PB1)
- net CE_MAG: now reaches U?.28 (PB2)
- net S1_control: now reaches U?.56 (PB4)
- net S1_control: now also J?.1 (Pin_1)
- net S2_control: now reaches U?.57 (PB5)
- net S2_control: now also J?.1 (Pin_1)
- new net +5V: J?.2 (Pin_2), J?.2 (Pin_2)
- new net OSC_IN: C?.1, Y?.1
- new net OSC_OUT: C?.1, Y?.2
Other:
- note added: "Ocillator for USB"
- note added: "SERVO INTERFACES"

Commit message: Continued pcb work
Parts:
- removed C? (x3): 100n, symbol Device:C
- removed C?: 33p, Capacitor_SMD:C_0402_1005Metric, symbol Device:C_Small
- added C1, C2: 15p, Capacitor_SMD:C_0805_2012Metric, symbol Device:C_Small
- added C3: 33p, Capacitor_SMD:C_0805_2012Metric, symbol Device:C_Small
- added C? (x3): 100nF, Capacitor_SMD:C_0603_1608Metric, symbol Device:C_Small
- added Y1: 32.768k, Crystal:Crystal_SMD_HC49-SD, symbol Device:Crystal
- C?: footprint Capacitor_SMD:C_0402_1005Metric -> Capacitor_SMD:C_0805_2012Metric; LCSC C1562 -> (none)
- J?: value (none) -> Conn_01x04; footprint (none) -> Connector_PinHeader_2.54mm:PinHeader_1x04_P2.54mm_Vertical
- U?: value (none) -> STM32F411RETx; footprint (none) -> Package_QFP:LQFP-64_10x10mm_P0.5mm
- Y?: value (none) -> 12MHz; footprint (none) -> Crystal:Crystal_SMD_HC49-SD
Connections:
- net +3V3: now also C?.1, C?.1
- net GND: now also C1.2, C2.2, C3.2, C?.2, C?.2, C?.2
- net OSC_IN: now also C1.1, Y1.1
- net OSC_OUT: now also C2.1, C3.1, Y1.2
- net at L?.2, U?.13 (VDDA): now also C?.1
- net CS_RF: now reaches U?.10 (PC2)
- net CS_SD: now reaches U?.11 (PC3)
- net SCK_RF: now reaches U?.34 (PB13)
- net MISO_RF: now reaches U?.35 (PB14)
- net MOSI_RF: now reaches U?.36 (PB15)
- net CLK_SD: now reaches U?.51 (PC10)
- net MISO_SD: now reaches U?.52 (PC11)
- net MOSI_SD: now reaches U?.53 (PC12)
- net RF_100: now reaches U?.8 (PC0)
- net RESET_RF: now reaches U?.9 (PC1)
Other:
- note added: "Boot"
- note added: "HSE oscillator"
- note added: "Helper circuits"
- note added: "LSE Oscillator"
- note added: "MCU protection"
- note added: "Oscillators"
- note added: "Reset"
- note added: "SWD interface"
- note added: "Servo interfaces"
- note added: "USB interface"
- note removed: "BOOT"
- note removed: "IC protection"
- note removed: "Ocillator for USB"
- note removed: "RESET"
- note removed: "SERVO INTERFACES"
- note removed: "SWD INTERFACE"
- note removed: "USB INTERFACE"
- moved on the sheet: C?, R?, SW?, Y?

Commit message: Schematic done I think
Parts:
- added C26: 4.7u, Capacitor_SMD:C_0603_1608Metric, symbol Device:C
- C22, C23: renamed from C?; footprint (none) -> Capacitor_SMD:C_0603_1608Metric
- L2: renamed from L?; footprint (none) -> Inductor_SMD:L_0805_2012Metric
- U6: renamed from U?; LCSC (none) -> C2827654
- U7: renamed from U?; LCSC (none) -> C94355
- Y1: footprint Crystal:Crystal_SMD_HC49-SD -> Crystal:Crystal_SMD_3215-2Pin_3.2x1.5mm; LCSC (none) -> C620155
- Y2: renamed from Y?; LCSC (none) -> C108151
- gave numbers to parts that had none: 10
Connections:
- net GND: now also C26.2
- net OSC_IN: now also U7.5 (PH0); no longer C1.1, Y1.1
- net OSC_OUT: now also U7.6 (PH1); no longer C2.1, Y1.2
- net OSC32_IN: now reaches U7.3 (PC14)
- net OSC32_IN: now also C1.1, Y1.1
- net at U7.30 (VCAP1): now also C26.1
- net OSC32_OUT: now reaches U7.4 (PC15)
- net OSC32_OUT: now also C2.1, Y1.2
Other:
- moved on the sheet: C1, C2, C21, C22, C23, C3, C?, L2, U7, Y1, Y2

Commit message: PCB done, pending review
Parts:
- Y2: footprint Crystal:Crystal_SMD_HC49-SD -> Crystal:Crystal_SMD_5032-2Pin_5.0x3.2mm; LCSC C108151 -> C251588
Other:
- moved on the sheet: C20, R11, SW2
Changed lines of the file:
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@@
   (junction (at 180.34 41.91) (diameter 0) (color 0 0 0 0)
   )
-  (junction (at 66.04 115.57) (diameter 0) (color 0 0 0 0)
+  (junction (at 67.31 115.57) (diameter 0) (color 0 0 0 0)
   )
   (junction (at 254 30.48) (diameter 0) (color 0 0 0 0)
@@
   (junction (at 35.56 118.11) (diameter 0) (color 0 0 0 0)
   )
-  (junction (at 68.58 125.73) (diameter 0) (color 0 0 0 0)
+  (junction (at 69.85 125.73) (diameter 0) (color 0 0 0 0)
   )
   (junction (at 248.92 121.92) (diameter 0) (color 0 0 0 0)
   )
-  (junction (at 68.58 115.57) (diameter 0) (color 0 0 0 0)
+  (junction (at 69.85 115.57) (diameter 0) (color 0 0 0 0)
   )
   (junction (at 243.84 121.92) (diameter 0) (color 0 0 0 0)
@@
     (stroke (width 0) (type default))
   )
-  (polyline (pts (xy 77.47 97.79) (xy 77.47 133.35))
+  (polyline (pts (xy 78.74 97.79) (xy 78.74 133.35))
     (stroke (width 0) (type default))
   )
@@
     (stroke (width 0) (type default))
   )
-  (wire (pts (xy 68.58 115.57) (xy 71.12 115.57))
+  (wire (pts (xy 69.85 115.57) (xy 72.39 115.57))
     (stroke (width 0) (type default))
   )
@@
     (stroke (width 0) (type default))
   )
-  (polyline (pts (xy 77.47 133.35) (xy 48.26 133.35))
+  (polyline (pts (xy 78.74 133.35) (xy 48.26 133.35))
     (stroke (width 0) (type default))
   )
@@
     (stroke (width 0) (type default))
   )
-  (wire (pts (xy 68.58 125.73) (xy 68.58 128.27))
+  (wire (pts (xy 69.85 125.73) (xy 69.85 128.27))
     (stroke (width 0) (type default))
   )
@@
     (stroke (width 0) (type default))
   )
-  (wire (pts (xy 66.04 115.57) (xy 68.58 115.57))
+  (wire (pts (xy 67.31 115.57) (xy 69.85 115.57))
     (stroke (width 0) (type default))
   )
@@
     (stroke (width 0) (type default))
   )
-  (polyline (pts (xy 48.26 97.79) (xy 77.47 97.79))
+  (polyline (pts (xy 48.26 97.79) (xy 78.74 97.79))
     (stroke (width 0) (type default))
   )
@@
     (stroke (width 0) (type default))
   )
-  (wire (pts (xy 68.58 123.19) (xy 68.58 125.73))
+  (wire (pts (xy 69.85 123.19) (xy 69.85 125.73))
     (stroke (width 0) (type default))
   )
@@
     (stroke (width 0) (type default))
   )
-  (wire (pts (xy 55.88 125.73) (xy 68.58 125.73))
+  (wire (pts (xy 57.15 125.73) (xy 69.85 125.73))
     (stroke (width 0) (type default))
   )
@@
     (stroke (width 0) (type default))
   )
-  (wire (pts (xy 55.88 115.57) (xy 66.04 115.57))
+  (wire (pts (xy 57.15 115.57) (xy 67.31 115.57))
     (stroke (width 0) (type default))
   )
@@
     (stroke (width 0) (type default))
   )
-  (wire (pts (xy 68.58 115.57) (xy 68.58 118.11))
+  (wire (pts (xy 69.85 115.57) (xy 69.85 118.11))
     (stroke (width 0) (type default))
   )
@@
     (stroke (width 0) (type default))
   )
-  (wire (pts (xy 66.04 115.57) (xy 66.04 113.03))
+  (wire (pts (xy 67.31 115.57) (xy 67.31 113.03))
     (stroke (width 0) (type default))
   )
@@
     (effects (font (size 1.27 1.27)) (justify right bottom))
   )
-  (label "NRST" (at 71.12 115.57 0) (fields_autoplaced)
+  (label "NRST" (at 72.39 115.57 0) (fields_autoplaced)
     (effects (font (size 1.27 1.27)) (justify left bottom))
   )
@@
       (effects (font (size 1.27 1.27)))
     )
-    (property "Footprint" "Crystal:Crystal_SMD_HC49-SD" (at 142.24 34.29 0)
-      (effects (font (size 1.27 1.27)) hide)
-    )
-    (property "Datasheet" "https://jlcpcb.com/partdetail/YangxingTech-X49SM12MSD2SI/C108151" (at 142.24 34.29 0)
-      (effects (font (size 1.27 1.27)) hide)
-    )
-    (property "LCSC" "C108151" (at 142.24 34.29 0)
+    (property "Footprint" "Crystal:Crystal_SMD_5032-2Pin_5.0x3.2mm" (at 142.24 34.29 0)
+      (effects (font (size 1.27 1.27)) hide)
+    )
+    (property "Datasheet" "https://jlcpcb.com/partdetail/247391-6I12000F20UCG/C251588" (at 142.24 34.29 0)
+      (effects (font (size 1.27 1.27)) hide)
+    )
+    (property "LCSC" "C251588" (at 142.24 34.29 0)
       (effects (font (size 1.27 1.27)) hide)
     )
@@
     )
   )
-  (symbol (lib_id "Device:R_Small") (at 66.04 110.49 180) (unit 1)
+  (symbol (lib_id "Device:R_Small") (at 67.31 110.49 180) (unit 1)
     (in_bom yes) (on_board yes) (dnp no)
-    (property "Reference" "R11" (at 61.595 109.22 0)
+    (property "Reference" "R11" (at 62.865 109.22 0)
       (effects (font (size 1.27 1.27)) (justify right))
     )
-    (property "Value" "10k" (at 61.595 111.76 0)
+    (property "Value" "10k" (at 62.865 111.76 0)
       (effects (font (size 1.27 1.27)) (justify right))
     )
-    (property "Footprint" "Resistor_SMD:R_0402_1005Metric" (at 66.04 110.49 0)
-      (effects (font (size 1.27 1.27)) hide)
-    )
-    (property "Datasheet" "~" (at 66.04 110.49 0)
+    (property "Footprint" "Resistor_SMD:R_0402_1005Metric" (at 67.31 110.49 0)
+      (effects (font (size 1.27 1.27)) hide)
+    )
+    (property "Datasheet" "~" (at 67.31 110.49 0)
       (effects (font (size 1.27 1.27)) hide)
     )
@@
     )
   )
-  (symbol (lib_id "power:+3.3V") (at 66.04 107.95 0) (unit 1)
+  (symbol (lib_id "power:+3.3V") (at 67.31 107.95 0) (unit 1)
     (in_bom yes) (on_board yes) (dnp no)
-    (property "Reference" "#PWR046" (at 66.04 111.76 0)
-      (effects (font (size 1.27 1.27)) hide)
-    )
-    (property "Value" "+3.3V" (at 66.04 104.14 0)
-      (effects (font (size 1.27 1.27)))
-    )
-    (property "Footprint" "" (at 66.04 107.95 0)
-      (effects (font (size 1.27 1.27)) hide)
-    )
-    (property "Datasheet" "" (at 66.04 107.95 0)
+    (property "Reference" "#PWR046" (at 67.31 111.76 0)
+      (effects (font (size 1.27 1.27)) hide)
+    )
+    (property "Value" "+3.3V" (at 67.31 104.14 0)
+      (effects (font (size 1.27 1.27)))
+    )
+    (property "Footprint" "" (at 67.31 107.95 0)
+      (effects (font (size 1.27 1.27)) hide)
+    )
+    (property "Datasheet" "" (at 67.31 107.95 0)
       (effects (font (size 1.27 1.27)) hide)
     )
@@
     )
   )
-  (symbol (lib_id "Device:C_Small") (at 68.58 120.65 0) (unit 1)
-    (in_bom yes) (on_board yes) (dnp no) (fields_autoplaced)
-    (property "Reference" "C20" (at 71.12 119.3862 0)
-      (effects (font (size 1.27 1.27)) (justify left))
-    )
-    (property "Value" "1u" (at 71.12 121.9262 0)
-      (effects (font (size 1.27 1.27)) (justify left))
-    )
-    (property "Footprint" "Capacitor_SMD:C_0402_1005Metric" (at 68.58 120.65 0)
-      (effects (font (size 1.27 1.27)) hide)
-    )
-    (property "Datasheet" "~" (at 68.58 120.65 0)
+  (symbol (lib_id "Device:C_Small") (at 69.85 120.65 0) (unit 1)
+    (in_bom yes) (on_board yes) (dnp no) (fields_autoplaced)
+    (property "Reference" "C20" (at 72.39 119.3862 0)
+      (effects (font (size 1.27 1.27)) (justify left))
+    )
+    (property "Value" "1u" (at 72.39 121.9262 0)
+      (effects (font (size 1.27 1.27)) (justify left))
+    )
+    (property "Footprint" "Capacitor_SMD:C_0402_1005Metric" (at 69.85 120.65 0)
+      (effects (font (size 1.27 1.27)) hide)
+    )
+    (property "Datasheet" "~" (at 69.85 120.65 0)
       (effects (font (size 1.27 1.27)) hide)
     )
@@
     )
   )
-  (symbol (lib_id "Switch:SW_Push") (at 55.88 120.65 90) (unit 1)
+  (symbol (lib_id "Switch:SW_Push") (at 57.15 120.65 90) (unit 1)
     (in_bom yes) (on_board yes) (dnp no)
-    (property "Reference" "SW2" (at 48.895 120.65 0)
-      (effects (font (size 1.27 1.27)))
-    )
-    (property "Value" "TS-1187A-B-A-B" (at 51.435 120.65 0)
-      (effects (font (size 1.27 1.27)))
-    )
-    (property "Footprint" "Button_Switch_SMD:SW_Push_1P1T_NO_CK_KSC6xxJ" (at 50.8 120.65 0)
-      (effects (font (size 1.27 1.27)) hide)
-    )
-    (property "Datasheet" "~" (at 50.8 120.65 0)
-      (effects (font (size 1.27 1.27)) hide)
-    )
-    (property "LCSC" "C318884" (at 55.88 120.65 0)
+    (property "Reference" "SW2" (at 50.165 120.65 0)
+      (effects (font (size 1.27 1.27)))
+    )
+    (property "Value" "TS-1187A-B-A-B" (at 52.705 120.65 0)
+      (effects (font (size 1.27 1.27)))
+    )
+    (property "Footprint" "Button_Switch_SMD:SW_Push_1P1T_NO_CK_KSC6xxJ" (at 52.07 120.65 0)
+      (effects (font (size 1.27 1.27)) hide)
+    )
+    (property "Datasheet" "~" (at 52.07 120.65 0)
+      (effects (font (size 1.27 1.27)) hide)
+    )
+    (property "LCSC" "C318884" (at 57.15 120.65 0)
       (effects (font (size 1.27 1.27)) hide)
     )
@@
     )
   )
-  (symbol (lib_id "power:GND") (at 68.58 128.27 0) (unit 1)
+  (symbol (lib_id "power:GND") (at 69.85 128.27 0) (unit 1)
     (in_bom yes) (on_board yes) (dnp no)
-    (property "Reference" "#PWR047" (at 68.58 134.62 0)
-      (effects (font (size 1.27 1.27)) hide)
-    )
-    (property "Value" "GND" (at 68.58 132.08 0)
-      (effects (font (size 1.27 1.27)))
-    )
-    (property "Footprint" "" (at 68.58 128.27 0)
-      (effects (font (size 1.27 1.27)) hide)
-    )
-    (property "Datasheet" "" (at 68.58 128.27 0)
-      (effects (font (size 1.27 1.27)) hide)
-    )
+    (property "Reference" "#PWR047" (at 69.85 134.62 0)
+      (effects (font (size 1.27 1.27)) hide)
+    )
+    (property "Value" "GND" (at 69.85 132.08 0)
+      (effects (font (size 1.27 1.27)))
+    )
+    (property "Footprint" "" (at 69.85 128.27 0)
+      (effects (font (size 1.27 1.27)) hide)
+    )
+    (property "Datasheet" "" (at 69.85 128.27 0)
+      (effects (font (size 1.27 1.27)) hide)
+    )

Commit message: Headaches
Parts:
- removed Y2: 12MHz, Crystal:Crystal_SMD_5032-2Pin_5.0x3.2mm, symbol Device:Crystal
- added Y2: 12MHz, Crystal:Crystal_SMD_5032-4Pin_5.0x3.2mm, symbol Device:Crystal_GND24
Connections:
- net GND: now also Y2.2, Y2.4
- net OSC_IN: now also Y2.1
- net OSC_OUT: now also Y2.3
Changed lines of the file:
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@@
+    (stroke (width 0) (type default))
+  )
+  (wire (pts (xy 142.24 25.4) (xy 148.59 25.4))
     (stroke (width 0) (type default))
   )
@@
     (stroke (width 0) (type default))
   )
+  (wire (pts (xy 148.59 25.4) (xy 148.59 26.67))
+    (stroke (width 0) (type default))
+  )
   (polyline (pts (xy 124.46 21.59) (xy 161.29 21.59))
     (stroke (width 0) (type default))
@@
   )
   (wire (pts (xy 246.38 120.65) (xy 246.38 121.92))
+    (stroke (width 0) (type default))
+  )
+  (wire (pts (xy 142.24 29.21) (xy 142.24 25.4))
     (stroke (width 0) (type default))
   )
@@
     (effects (font (size 2.3 2.3) italic) (justify left bottom))
   )
-  (text "HSE oscillator\n" (at 129.54 30.48 0)
+  (text "HSE oscillator\n" (at 151.13 30.48 0)
     (effects (font (size 0.8 0.8)) (justify left bottom))
   )
@@
         (path "/e63e39d7-6ac0-4ffd-8aa3-1841a4541b55/708c8a34-f258-4554-8b50-7818f1e46fec"
           (reference "#PWR054") (unit 1)
-        )
-      )
-    )
-  )
-  (symbol (lib_id "Device:Crystal") (at 142.24 34.29 0) (unit 1)
-    (in_bom yes) (on_board yes) (dnp no) (fields_autoplaced)
-    (property "Reference" "Y2" (at 142.24 27.94 0)
-      (effects (font (size 1.27 1.27)))
-    )
-    (property "Value" "12MHz" (at 142.24 30.48 0)
-      (effects (font (size 1.27 1.27)))
-    )
-    (property "Footprint" "Crystal:Crystal_SMD_5032-2Pin_5.0x3.2mm" (at 142.24 34.29 0)
-      (effects (font (size 1.27 1.27)) hide)
-    )
-    (property "Datasheet" "https://jlcpcb.com/partdetail/247391-6I12000F20UCG/C251588" (at 142.24 34.29 0)
-      (effects (font (size 1.27 1.27)) hide)
-    )
-    (property "LCSC" "C251588" (at 142.24 34.29 0)
-      (effects (font (size 1.27 1.27)) hide)
-    )
-    (pin "1")
-    (pin "2")
-    (instances
-      (project "neptune"
-        (path "/e63e39d7-6ac0-4ffd-8aa3-1841a4541b55/708c8a34-f258-4554-8b50-7818f1e46fec"
-          (reference "Y2") (unit 1)
         )
       )
@@
         (path "/e63e39d7-6ac0-4ffd-8aa3-1841a4541b55/708c8a34-f258-4554-8b50-7818f1e46fec"
           (reference "C1") (unit 1)
+        )
+      )
+    )
+  )
+  (symbol (lib_id "Device:Crystal_GND24") (at 142.24 34.29 0) (unit 1)
+    (in_bom yes) (on_board yes) (dnp no)
+    (property "Reference" "Y2" (at 135.89 27.94 0)
+      (effects (font (size 1.27 1.27)))
+    )
+    (property "Value" "12MHz" (at 135.89 30.48 0)
+      (effects (font (size 1.27 1.27)))
+    )
+    (property "Footprint" "Crystal:Crystal_SMD_5032-4Pin_5.0x3.2mm" (at 142.24 34.29 0)
+      (effects (font (size 1.27 1.27)) hide)
+    )
+    (property "Datasheet" "https://www.digikey.com.au/en/products/detail/ecs-inc/ECS-120-20-30B-TR/813205" (at 142.24 34.29 0)
+      (effects (font (size 1.27 1.27)) hide)
+    )
+    (pin "1")
+    (pin "2")
+    (pin "3")
+    (pin "4")
+    (instances
+      (project "neptune"
+        (path "/e63e39d7-6ac0-4ffd-8aa3-1841a4541b55/708c8a34-f258-4554-8b50-7818f1e46fec"
+          (reference "Y2") (unit 1)
         )
       )
@@
     )
   )
+  (symbol (lib_id "power:GND") (at 142.24 39.37 0) (unit 1)
+    (in_bom yes) (on_board yes) (dnp no) (fields_autoplaced)
+    (property "Reference" "#PWR065" (at 142.24 45.72 0)
+      (effects (font (size 1.27 1.27)) hide)
+    )
+    (property "Value" "GND" (at 142.24 44.45 0)
+      (effects (font (size 1.27 1.27)))
+    )
+    (property "Footprint" "" (at 142.24 39.37 0)
+      (effects (font (size 1.27 1.27)) hide)
+    )
+    (property "Datasheet" "" (at 142.24 39.37 0)
+      (effects (font (size 1.27 1.27)) hide)
+    )
+    (pin "1")
+    (instances
+      (project "neptune"
+        (path "/e63e39d7-6ac0-4ffd-8aa3-1841a4541b55/708c8a34-f258-4554-8b50-7818f1e46fec"
+          (reference "#PWR065") (unit 1)
+        )
+      )
+    )
+  )
   (symbol (lib_id "Device:R_Small") (at 67.31 110.49 180) (unit 1)
     (in_bom yes) (on_board yes) (dnp no)
@@
   )
   (symbol (lib_id "Device:C_Small") (at 135.89 39.37 0) (unit 1)
-    (in_bom yes) (on_board yes) (dnp no) (fields_autoplaced)
-    (property "Reference" "C21" (at 138.43 38.1062 0)
-      (effects (font (size 1.27 1.27)) (justify left))
-    )
-    (property "Value" "33p" (at 138.43 40.6462 0)
+    (in_bom yes) (on_board yes) (dnp no)
+    (property "Reference" "C21" (at 129.54 38.1 0)
+      (effects (font (size 1.27 1.27)) (justify left))
+    )
+    (property "Value" "33p" (at 129.54 40.64 0)
       (effects (font (size 1.27 1.27)) (justify left))
     )
@@
         )
       )
+    )
+  )
+  (symbol (lib_id "power:GND") (at 148.59 26.67 0) (unit 1)
+    (in_bom yes) (on_board yes) (dnp no) (fields_autoplaced)
+    (property "Reference" "#PWR066" (at 148.59 33.02 0)
+      (effects (font (size 1.27 1.27)) hide)
+    )
+    (property "Value" "GND" (at 148.59 31.75 0)
+      (effects (font (size 1.27 1.27)))
+    )
+    (property "Footprint" "" (at 148.59 26.67 0)
+      (effects (font (size 1.27 1.27)) hide)
+    )
+    (property "Datasheet" "" (at 148.59 26.67 0)
+      (effects (font (size 1.27 1.27)) hide)
+    )
+    (pin "1")
+    (instances
+      (project "neptune"
+        (path "/e63e39d7-6ac0-4ffd-8aa3-1841a4541b55/708c8a34-f258-4554-8b50-7818f1e46fec"
+          (reference "#PWR066") (unit 1)
+        )
+      )
