File: neptune-flight-computer/neptune.kicad_pcb (KiCad board)
At the start: 4 copper layers, 39 x 67.2 mm, 69 parts, among them J1 THD2528-11SD-GF, J2 Conn_01x02, J3 Conn_Coaxial, J4 USB_B_Micro, J5 Conn_01x04, J6 Conn_01x04, J7 Conn_01x04, Q1 Si2301-TP, Q2 AO3401A, SW1 TS-1187A-B-A-B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

Commit message: Fixed corrupt PCB file, updated schematic
Parts:
- R1: value 56k -> 30k
- R3: value 30k -> 56k
- R4: value 10k -> 30k
Connections:
- C10 pad 1: +3.3V -> +3V3
- C22 pad 1: +3.3V -> +3V3
- C23 pad 1: +3.3V -> +3V3
- C24 pad 1: +3.3V -> +3V3
- C25 pad 1: +3.3V -> +3V3
- C9 pad 1: +3.3V -> +3V3
- J5 pad 1: +3.3V -> +3V3
- L2 pad 1: +3.3V -> +3V3
- R11 pad 2: +3.3V -> +3V3
- SW1 pad 2: +3.3V -> +3V3
- U7 pad 1: +3.3V -> +3V3
- U7 pad 19: +3.3V -> +3V3
- U7 pad 32: +3.3V -> +3V3
- U7 pad 48: +3.3V -> +3V3
- U7 pad 64: +3.3V -> +3V3
- U8 pad 13: +3.3V -> +3V3
- U8 pad 3: +3.3V -> +3V3
Routing:
- net +3.3V: track 58.5 -> 34.9 mm
- net +3V3: track 0.00 -> 23.6 mm
